File: KiCad/sensing unit1/sensing unit1.sch (KiCad schematic (older format))
At the start: 25 parts, among them J1 Conn_01x03_Male, J2 Conn_01x03_Male, J3 Conn_01x03_Male, J4 Conn_01x03_Male, J5 Conn_01x03_Male, U1 LM358, U2 LM358

Commit message: .
.
Parts:
- added R?: 500k, Resistor_THT:R_Axial_DIN0309_L9.0mm_D3.2mm_P12.70mm_Horizontal, symbol Device:R
- R10: value 500 -> 0
- R11: value 330 -> 560
- R5, R6: value 25k -> 56k
Connections:
- net GND: now also R?.2
- net at D5.1 (K), R9.2, U2.3 (+): now also R?.1
Other:
- note added: "Vout =56*(LM35 voltage- OFFSET VOLTAGE) - Vdiode_on\n0<Vout<8.8V\nOFFSET_VOLTAGE = Voltage of LM35 at 24C + Viode_on/25.\n\nVout (C) = 0.56*(C-24), \nat 24C, Vout = 0V & at 40C, vout = 9V"
- note removed: "Vout = 25*(LM35 voltage- OFFSET VOLTAGE) - Vdiode_on\n0<Vout<4.7V\nOFFSET_VOLTAGE = Voltage of LM35 at 24C + Viode_on/25.\n\nVout (C) = 0.25*(C-24), \nat 24C, Vout = 0V & at 40C, vout = 4V"
Changed lines of the file:
@@
 P 4150 3850
 F 0 "R6" V 3943 3850 50  0000 C CNN
-F 1 "25k" V 4034 3850 50  0000 C CNN
+F 1 "56k" V 4034 3850 50  0000 C CNN
 F 2 "Resistor_THT:R_Axial_DIN0309_L9.0mm_D3.2mm_P12.70mm_Horizontal" V 4080 3850 50  0001 C CNN
 F 3 "~" H 4150 3850 50  0001 C CNN
@@
 P 3900 2650
 F 0 "R5" H 3970 2696 50  0000 L CNN
-F 1 "25k" H 3970 2605 50  0000 L CNN
+F 1 "56k" H 3970 2605 50  0000 L CNN
 F 2 "Resistor_THT:R_Axial_DIN0309_L9.0mm_D3.2mm_P12.70mm_Horizontal" V 3830 2650 50  0001 C CNN
 F 3 "~" H 3900 2650 50  0001 C CNN
@@
 	0    -1   -1   0
 $EndComp
-$Comp
-L Device:D_Zener D5
-U 1 1 61E731BF
-P 6250 3550
-F 0 "D5" V 6204 3630 50  0000 L CNN
-F 1 "4.7V" V 6295 3630 50  0000 L CNN
-F 2 "Diode_THT:D_A-405_P12.70mm_Horizontal" H 6250 3550 50  0001 C CNN
-F 3 "~" H 6250 3550 50  0001 C CNN
-	1    6250 3550
-	0    1    1    0
-$EndComp
 Text GLabel 6250 3850 3    50   Input ~ 0
 GND
@@
 Connection ~ 6250 3250
 Wire Wire Line
-	6250 3250 7100 3250
+	6250 3250 6600 3250
 Wire Wire Line
 	6950 3450 7100 3450
@@
 P 8100 5250
 F 0 "R10" H 8170 5296 50  0000 L CNN
-F 1 "500" H 8170 5205 50  0000 L CNN
+F 1 "0" H 8170 5205 50  0000 L CNN
 F 2 "Resistor_THT:R_Axial_DIN0309_L9.0mm_D3.2mm_P12.70mm_Horizontal" V 8030 5250 50  0001 C CNN
 F 3 "~" H 8100 5250 50  0001 C CNN
@@
 P 8100 5600
 F 0 "R11" H 8170 5646 50  0000 L CNN
-F 1 "330" H 8170 5555 50  0000 L CNN
+F 1 "560" H 8170 5555 50  0000 L CNN
 F 2 "Resistor_THT:R_Axial_DIN0309_L9.0mm_D3.2mm_P12.70mm_Horizontal" V 8030 5600 50  0001 C CNN
 F 3 "~" H 8100 5600 50  0001 C CNN
@@
 	6800 2700 7850 2700
 Text Notes 8750 3550 0    50   ~ 0
-Vout = 25*(LM35 voltage- OFFSET VOLTAGE) - Vdiode_on\n0<Vout<4.7V\nOFFSET_VOLTAGE = Voltage of LM35 at 24C + Viode_on/25.\n\nVout (C) = 0.25*(C-24), \nat 24C, Vout = 0V & at 40C, vout = 4V
+Vout =56*(LM35 voltage- OFFSET VOLTAGE) - Vdiode_on\n0<Vout<8.8V\nOFFSET_VOLTAGE = Voltage of LM35 at 24C + Viode_on/25.\n\nVout (C) = 0.56*(C-24), \nat 24C, Vout = 0V & at 40C, vout = 9V
 Wire Notes Line
 	11050 3050 11050 3600
@@
 EndData
 $EndBitmap
+$Comp
+L Device:D_Zener D5
+U 1 1 61E731BF
+P 6250 3550
+F 0 "D5" V 6204 3630 50  0000 L CNN
+F 1 "4.7V" V 6295 3630 50  0000 L CNN
+F 2 "Diode_THT:D_A-405_P12.70mm_Horizontal" H 6250 3550 50  0001 C CNN
+F 3 "~" H 6250 3550 50  0001 C CNN
+	1    6250 3550
+	0    1    1    0
+$EndComp
+$Comp
+L Device:R R?
+U 1 1 61E78901
+P 6600 3550
+F 0 "R?" V 6807 3550 50  0000 C CNN
+F 1 "500k" V 6716 3550 50  0000 C CNN
+F 2 "Resistor_THT:R_Axial_DIN0309_L9.0mm_D3.2mm_P12.70mm_Horizontal" V 6530 3550 50  0001 C CNN
+F 3 "~" H 6600 3550 50  0001 C CNN
+	1    6600 3550
+	1    0    0    -1
+$EndComp
+Text GLabel 6600 3850 3    50   Input ~ 0
+GND
+Wire Wire Line
+	6600 3850 6600 3700
+Wire Wire Line
+	6600 3400 6600 3250
+Connection ~ 6600 3250
+Wire Wire Line
+	6600 3250 7100 3250
 $EndSCHEMATC

Commit message: Final report is finished
.
Parts:
- added D1: D, Diode_THT:D_A-405_P12.70mm_Horizontal, symbol Device:D
- added D?: GREEN, LED_THT:LED_D3.0mm_FlatTop, symbol Device:LED
- added D?: BLUE, LED_THT:LED_D3.0mm_FlatTop, symbol Device:LED
- added R1: 3k, Resistor_THT:R_Axial_DIN0309_L9.0mm_D3.2mm_P12.70mm_Horizontal, symbol Device:R
- added R2: 50k, Resistor_THT:R_Axial_DIN0309_L9.0mm_D3.2mm_P12.70mm_Horizontal, symbol Device:R
- added R3 (x2): 1k, Resistor_THT:R_Axial_DIN0309_L9.0mm_D3.2mm_P12.70mm_Horizontal, symbol Device:R
- added R4 (x2): 56k, Resistor_THT:R_Axial_DIN0309_L9.0mm_D3.2mm_P12.70mm_Horizontal, symbol Device:R
- added R5: 10k, Resistor_THT:R_Axial_DIN0309_L9.0mm_D3.2mm_P12.70mm_Horizontal, symbol Device:R
- added R6: 500k, Resistor_THT:R_Axial_DIN0309_L9.0mm_D3.2mm_P12.70mm_Horizontal, symbol Device:R
- added R7: 560, Resistor_THT:R_Axial_DIN0309_L9.0mm_D3.2mm_P12.70mm_Horizontal, symbol Device:R
- added R8, R9: 1.2k, Resistor_THT:R_Axial_DIN0309_L9.0mm_D3.2mm_P12.70mm_Horizontal, symbol Device:R
- added RED_LED_Temperature: RED, LED_THT:LED_D3.0mm_FlatTop, symbol Device:LED
- added R_POT: 5k, Potentiometer_THT:Potentiometer_Alps_RK163_Single_Horizontal, symbol Device:R_POT
- added U?: OPAMP, Package_DIP:DIP-8_W7.62mm, symbol Amplifier_Operational:LM358
- added U? (x2): LM358, Package_DIP:DIP-8_W7.62mm, symbol Amplifier_Operational:LM358
- added Z1: 5.1V, Diode_THT:D_A-405_P12.70mm_Horizontal, symbol Device:D_Zener
- added Z2: 4.7V, Diode_THT:D_A-405_P12.70mm_Horizontal, symbol Device:D_Zener
- D5: value 4.7V -> 9V
- renumbered RV1 to R_POT
Connections:
- net -12V: now also D?.1 (K)
- net 12V: now also D?.2 (A), R1.1
- net GND: now also R4.1, R6.2, R7.2, R8.1, R9.1, R_POT.1, Z1.2 (A), Z2.2 (A)
- net LM35: now also R3.2
- new net: R1.2, R2.1, Z1.1 (K)
- new net: R2.2, R_POT.3
- new net: R3.1, R4.2, U?.5 (+)
- new net: R3.1, R4.2, U?.6 (-)
- new net: D1.1 (K), R5.1
- new net: R7.1, RED_LED_Temperature.1 (K), U?.6 (-)
- new net: RED_LED_Temperature.2 (A), U?.7
- new net: D?.1 (K), R8.2
- new net: D?.2 (A), R9.2
- new net Amplified_Signal: R4.1, U?.7
- new net Amplified_signal: D1.2 (A)
- new net Offset_voltage: R3.2, R_POT.2
- new net Vsensing: U?.1, U?.2 (-), U?.5 (+)
- new net Vsensing_clipped: R5.2, R6.1, U?.3 (+), Z2.1 (K)
Other:
- moved on the sheet: D1, D2, D3, D4, D5, D6, J1, J2, J3, J4, J5, R1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
